File: 7SegLED_Array.kicad_pcb (KiCad board)
At the start: 2 copper layers, 129.5 x 69.9 mm, 12 parts, among them J1 Conn_02x08_Odd_Even, Q1 RT1P137P, Q2 RT1P137P, Q3 RT1P137P, Q4 RT1P137P, U1 TBD62083A, U2 7SEGMENT_CA, U3 7SEGMENT_CA, U4 7SEGMENT_CA, U5 7SEGMENT_CA

Commit message: edit
Parts:
- RN1: footprint Housings_DIP:DIP-16_W8.89mm_SMDSocket_LongPads -> Resistors_SMD:R_Array_Convex_8x0602
- moved Q3 7.22 mm to (225.7, 29.2), turned to 90 degrees
- moved Q4 6.84 mm to (237.5, 29.2), turned to 90 degrees
- moved Q2 6.48 mm to (210.8, 29.2), turned to 90 degrees
- moved Q1 6.36 mm to (197.2, 29.2), turned to 90 degrees
Routing:
- net +5V: track 110.7 -> 0.00 mm
- net DIG4: track 84.7 -> 0.00 mm, vias 1 -> 0
- net Net-(RN1-Pad11): track 79.0 -> 0.00 mm
- net DIG3: track 77.7 -> 0.00 mm
- net Net-(RN1-Pad10): track 77.0 -> 0.00 mm
- net Net-(RN1-Pad14): track 67.5 -> 0.00 mm
- net Net-(RN1-Pad13): track 67.4 -> 0.00 mm
- net Net-(RN1-Pad15): track 67.4 -> 0.00 mm
- net Net-(RN1-Pad16): track 64.6 -> 0.00 mm
- net Net-(R1-Pad1): track 60.0 -> 0.00 mm
- net DIG2: track 57.3 -> 0.00 mm
- net Net-(RN1-Pad12): track 55.5 -> 0.41 mm
- net DIG1: track 47.7 -> 0.00 mm
- net Net-(Q1-Pad2): track 32.1 -> 0.00 mm, vias 1 -> 0
- net Net-(Q4-Pad2): track 25.7 -> 0.00 mm
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