File: 7SegLED_Array.sch (KiCad schematic (older format))
At the start: 12 parts, among them J1 Conn_02x08_Odd_Even, Q1 RT1P137P, Q2 RT1P137P, Q3 RT1P137P, Q4 RT1P137P, U1 TBD62083A, U2 7SEGMENT_CA, U3 7SEGMENT_CA, U4 7SEGMENT_CA, U5 7SEGMENT_CA

Commit message: KiCAD 5
Parts:
- J1: symbol Conn_02x08_Odd_Even -> 7SegLED_Array-rescue:Conn_02x08_Odd_Even
- Q1, Q2, Q3, Q4: symbol RT1P137P -> RT1P137P:RT1P137P
- R1: symbol R_Small -> Device:R_Small
- RN1: symbol R_Pack08 -> Device:R_Pack08
- U1: symbol TBD62083A -> TBD62083A:TBD62083A
- U2, U3, U4, U5: symbol 7SEGMENT_CA -> 7SegLED_Array-rescue:7SEGMENT_CA
Changed lines of the file:
@@
-EESchema Schematic File Version 2
-LIBS:7SegLED_Array-rescue
-LIBS:power
-LIBS:device
-LIBS:transistors
-LIBS:conn
-LIBS:linear
-LIBS:regul
-LIBS:74xx
-LIBS:cmos4000
-LIBS:adc-dac
-LIBS:memory
-LIBS:xilinx
-LIBS:microcontrollers
-LIBS:dsp
-LIBS:microchip
-LIBS:analog_switches
-LIBS:motorola
-LIBS:texas
-LIBS:intel
-LIBS:audio
-LIBS:interface
-LIBS:digital-audio
-LIBS:philips
-LIBS:display
-LIBS:cypress
-LIBS:siliconi
-LIBS:opto
-LIBS:atmel
-LIBS:contrib
-LIBS:valves
-LIBS:RT1P137P
-LIBS:TBD62083A
-LIBS:CSD-5622D
+EESchema Schematic File Version 4
 LIBS:7SegLED_Array-cache
-EELAYER 25 0
+EELAYER 26 0
 EELAYER END
 $Descr A4 11693 8268
@@
 $EndDescr
 $Comp
-L 7SEGMENT_CA U2
+L 7SegLED_Array-rescue:7SEGMENT_CA U2
 U 1 1 5AB3072E
 P 4200 2750
@@
 $EndComp
 $Comp
-L 7SEGMENT_CA U3
+L 7SegLED_Array-rescue:7SEGMENT_CA U3
 U 1 1 5AB30795
 P 5350 2750
@@
 $EndComp
 $Comp
-L 7SEGMENT_CA U4
+L 7SegLED_Array-rescue:7SEGMENT_CA U4
 U 1 1 5AB307C4
 P 6500 2750
@@
 $EndComp
 $Comp
-L 7SEGMENT_CA U5
+L 7SegLED_Array-rescue:7SEGMENT_CA U5
 U 1 1 5AB30801
 P 7650 2750
@@
 $EndComp
 $Comp
-L +5V #PWR7
+L power:+5V #PWR7
 U 1 1 5AB32335
 P 4300 1650
@@
 $EndComp
 $Comp
-L +5V #PWR8
+L power:+5V #PWR8
 U 1 1 5AB32359
 P 5450 1650
@@
 $EndComp
 $Comp
-L +5V #PWR9
+L power:+5V #PWR9
 U 1 1 5AB3237D
 P 6600 1650
@@
 $EndComp
 $Comp
-L +5V #PWR10
+L power:+5V #PWR10
 U 1 1 5AB32609
 P 7750 1650
@@
 DIG4
 $Comp
-L R_Pack08 RN1
+L Device:R_Pack08 RN1
 U 1 1 5AB34DA5
 P 3500 3650
@@
 $EndComp
 $Comp
-L RT1P137P Q4
+L RT1P137P:RT1P137P Q4
 U 1 1 5AB355D0
 P 7650 1950
@@
 $EndComp
 $Comp
-L RT1P137P Q3
+L RT1P137P:RT1P137P Q3
 U 1 1 5AB35615
 P 6500 1950
@@
 $EndComp
 $Comp
-L RT1P137P Q2
+L RT1P137P:RT1P137P Q2
 U 1 1 5AB35638
 P 5350 1950
@@
 $EndComp
 $Comp
-L RT1P137P Q1
+L RT1P137P:RT1P137P Q1
 U 1 1 5AB3593C
 P 4200 1950
@@
 $EndComp
 $Comp
-L TBD62083A U1
+L TBD62083A:TBD62083A U1
 U 1 1 5AB388E6
 P 2750 3550
@@
 SEG_DP
 $Comp
-L GND #PWR3
+L power:GND #PWR3
 U 1 1 5AB39469
 P 2750 4350
@@
 $EndComp
 $Comp
-L +5V #PWR5
+L power:+5V #PWR5
 U 1 1 5AB39C54
 P 3250 3050
@@
 $EndComp
 $Comp
-L PWR_FLAG #FLG1
+L power:PWR_FLAG #FLG1
 U 1 1 5AB3319B
 P 2750 1350
@@
 $EndComp
 $Comp
-L PWR_FLAG #FLG2
+L power:PWR_FLAG #FLG2
 U 1 1 5AB331C3
 P 3150 1450
@@
 $EndComp
 $Comp
-L +5V #PWR4
+L power:+5V #PWR4
 U 1 1 5AB331EB
 P 3150 1350
@@
 $EndComp
 $Comp
-L GND #PWR2
+L power:GND #PWR2
 U 1 1 5AB33213
 P 2750 1450
@@
 	3800 3150 3800 3250
 Wire Wire Line
-	3700 3250 7250 3250
+	3700 3250 3800 3250
 Wire Wire Line
 	7250 3250 7250 3150
@@
 	3900 3150 3900 3350
 Wire Wire Line
-	3700 3350 7350 3350
+	3700 3350 3900 3350
 Wire Wire Line
 	7350 3350 7350 3150
@@
 	4000 3150 4000 3450
 Wire Wire Line
-	3700 3450 7450 3450
+	3700 3450 4000 3450
 Wire Wire Line
 	7450 3450 7450 3150
@@
 	4100 3150 4100 3550
 Wire Wire Line
-	3700 3550 7550 3550
+	3700 3550 4100 3550
 Wire Wire Line
 	7550 3550 7550 3150
@@
 	4200 3150 4200 3650
 Wire Wire Line
-	3700 3650 7650 3650
+	3700 3650 4200 3650
 Wire Wire Line
 	7650 3650 7650 3150
@@
 	4300 3150 4300 3750
 Wire Wire Line
-	3700 3750 7750 3750
+	3700 3750 4300 3750
 Wire Wire Line
 	7750 3750 7750 3150
@@
 	4400 3150 4400 3850
 Wire Wire Line
-	3700 3850 7850 3850
+	3700 3850 4400 3850
 Wire Wire Line
 	7850 3850 7850 3150
@@
 	4300 1750 4300 1650
 Wire Wire Line
-	4300 2150 4300 2350
-Wire Wire Line
-	5450 2150 5450 2350
+	4300 2150 4300 2250
+Wire Wire Line
+	5450 2150 5450 2250
 Wire Wire Line
 	5450 1750 5450 1650
 Wire Wire Line
-	6600 2150 6600 2350
-Wire Wire Line
-	7750 2150 7750 2350
+	6600 2150 6600 2250
+Wire Wire Line
+	7750 2150 7750 2250
 Wire Wire Line
 	7750 1750 7750 1650
@@
 	3150 1350 3150 1450
 $Comp
-L GND #PWR1
+L power:GND #PWR1
 U 1 1 5AB3438D
 P 2000 2650
@@
 $EndComp
 $Comp
-L +5V #PWR6
+L power:+5V #PWR6
 U 1 1 5AB343B7
 P 3450 2550
@@
 	3450 2600 3450 2550
 $Comp
-L Conn_02x08_Odd_Even J1
+L 7SegLED_Array-rescue:Conn_02x08_Odd_Even J1
 U 1 1 5AB344E7
 P 2700 2300
@@
 NoConn ~ 2900 2500
 $Comp
-L R_Small R1
+L Device:R_Small R1
 U 1 1 5AB3542C
 P 3950 3950
@@
 $EndComp
 Wire Wire Line
-	8050 3950 4050 3950
+	8050 3950 6900 3950
 Wire Wire Line
 	3850 3950 3700 3950
@@
 Connection ~ 5750 3950
 Connection ~ 4600 3950
+Wire Wire Line
+	4950 3250 6100 3250
+Wire Wire Line
+	5050 3350 6200 3350
+Wire Wire Line
+	5150 3450 6300 3450
+Wire Wire Line
+	5250 3550 6400 3550
+Wire Wire Line
+	5350 3650 6500 3650
+Wire Wire Line
+	5450 3750 6600 3750
+Wire Wire Line
+	5550 3850 6700 3850
+Wire Wire Line
+	6100 3250 7250 3250
+Wire Wire Line
+	6200 3350 7350 3350
+Wire Wire Line
+	6300 3450 7450 3450
+Wire Wire Line
+	6400 3550 7550 3550
+Wire Wire Line
+	6500 3650 7650 3650
+Wire Wire Line
+	6600 3750 7750 3750
+Wire Wire Line
+	6700 3850 7850 3850
+Wire Wire Line
+	3800 3250 4950 3250
+Wire Wire Line
+	3900 3350 5050 3350
+Wire Wire Line
+	4000 3450 5150 3450
+Wire Wire Line
+	4100 3550 5250 3550
+Wire Wire Line
+	4200 3650 5350 3650
+Wire Wire Line
+	4300 3750 5450 3750
+Wire Wire Line
+	4400 3850 5550 3850
+Wire Wire Line
+	4300 2250 4300 2350
+Wire Wire Line
+	5450 2250 5450 2350
+Wire Wire Line
+	6600 2250 6600 2350
+Wire Wire Line
+	7750 2250 7750 2350
+Wire Wire Line
+	6900 3950 5750 3950
+Wire Wire Line
+	5750 3950 4600 3950
+Wire Wire Line
+	4600 3950 4050 3950
 $EndSCHEMATC

Commit message: edit
Parts:
- RN1: value 470 -> 220
Changed lines of the file:
@@
 $EndComp
 $Comp
-L power:+5V #PWR7
+L power:+5V #PWR07
 U 1 1 5AB32335
 P 4300 1650
-F 0 "#PWR7" H 4300 1500 50  0001 C CNN
+F 0 "#PWR07" H 4300 1500 50  0001 C CNN
 F 1 "+5V" H 4300 1790 50  0000 C CNN
 F 2 "" H 4300 1650 50  0001 C CNN
@@
 $EndComp
 $Comp
-L power:+5V #PWR8
+L power:+5V #PWR08
 U 1 1 5AB32359
 P 5450 1650
-F 0 "#PWR8" H 5450 1500 50  0001 C CNN
+F 0 "#PWR08" H 5450 1500 50  0001 C CNN
 F 1 "+5V" H 5450 1790 50  0000 C CNN
 F 2 "" H 5450 1650 50  0001 C CNN
@@
 $EndComp
 $Comp
-L power:+5V #PWR9
+L power:+5V #PWR09
 U 1 1 5AB3237D
 P 6600 1650
-F 0 "#PWR9" H 6600 1500 50  0001 C CNN
+F 0 "#PWR09" H 6600 1500 50  0001 C CNN
 F 1 "+5V" H 6600 1790 50  0000 C CNN
 F 2 "" H 6600 1650 50  0001 C CNN
@@
 $EndComp
 $Comp
-L power:+5V #PWR10
+L power:+5V #PWR010
 U 1 1 5AB32609
 P 7750 1650
-F 0 "#PWR10" H 7750 1500 50  0001 C CNN
+F 0 "#PWR010" H 7750 1500 50  0001 C CNN
 F 1 "+5V" H 7750 1790 50  0000 C CNN
 F 2 "" H 7750 1650 50  0001 C CNN
@@
 P 3500 3650
 F 0 "RN1" V 3000 3650 50  0000 C CNN
-F 1 "470" V 3900 3650 50  0000 C CNN
+F 1 "220" V 3900 3650 50  0000 C CNN
 F 2 "Resistors_SMD:R_Array_Convex_8x0602" V 3975 3650 50  0001 C CNN
 F 3 "" H 3500 3650 50  0001 C CNN
@@
 SEG_DP
 $Comp
-L power:GND #PWR3
+L power:GND #PWR03
 U 1 1 5AB39469
 P 2750 4350
-F 0 "#PWR3" H 2750 4100 50  0001 C CNN
+F 0 "#PWR03" H 2750 4100 50  0001 C CNN
 F 1 "GND" H 2750 4200 50  0000 C CNN
 F 2 "" H 2750 4350 50  0001 C CNN
@@
 $EndComp
 $Comp
-L power:+5V #PWR5
+L power:+5V #PWR05
 U 1 1 5AB39C54
 P 3250 3050
-F 0 "#PWR5" H 3250 2900 50  0001 C CNN
+F 0 "#PWR05" H 3250 2900 50  0001 C CNN
 F 1 "+5V" H 3250 3190 50  0000 C CNN
 F 2 "" H 3250 3050 50  0001 C CNN
@@
 $EndComp
 $Comp
-L power:PWR_FLAG #FLG1
+L power:PWR_FLAG #FLG01
 U 1 1 5AB3319B
 P 2750 1350
-F 0 "#FLG1" H 2750 1425 50  0001 C CNN
+F 0 "#FLG01" H 2750 1425 50  0001 C CNN
 F 1 "PWR_FLAG" H 2750 1500 50  0000 C CNN
 F 2 "" H 2750 1350 50  0001 C CNN
@@
 $EndComp
 $Comp
-L power:PWR_FLAG #FLG2
+L power:PWR_FLAG #FLG02
 U 1 1 5AB331C3
 P 3150 1450
-F 0 "#FLG2" H 3150 1525 50  0001 C CNN
+F 0 "#FLG02" H 3150 1525 50  0001 C CNN
 F 1 "PWR_FLAG" H 3150 1600 50  0000 C CNN
 F 2 "" H 3150 1450 50  0001 C CNN
@@
 $EndComp
 $Comp
-L power:+5V #PWR4
+L power:+5V #PWR04
 U 1 1 5AB331EB
 P 3150 1350
-F 0 "#PWR4" H 3150 1200 50  0001 C CNN
+F 0 "#PWR04" H 3150 1200 50  0001 C CNN
 F 1 "+5V" H 3150 1490 50  0000 C CNN
 F 2 "" H 3150 1350 50  0001 C CNN
@@
 $EndComp
 $Comp
-L power:GND #PWR2
+L power:GND #PWR02
 U 1 1 5AB33213
 P 2750 1450
-F 0 "#PWR2" H 2750 1200 50  0001 C CNN
+F 0 "#PWR02" H 2750 1200 50  0001 C CNN
 F 1 "GND" H 2750 1300 50  0000 C CNN
 F 2 "" H 2750 1450 50  0001 C CNN
@@
 	3150 1350 3150 1450
 $Comp
-L power:GND #PWR1
+L power:GND #PWR01
 U 1 1 5AB3438D
 P 2000 2650
-F 0 "#PWR1" H 2000 2400 50  0001 C CNN
+F 0 "#PWR01" H 2000 2400 50  0001 C CNN
 F 1 "GND" H 2000 2500 50  0000 C CNN
 F 2 "" H 2000 2650 50  0001 C CNN
@@
 $EndComp
 $Comp
-L power:+5V #PWR6
+L power:+5V #PWR06
 U 1 1 5AB343B7
 P 3450 2550
-F 0 "#PWR6" H 3450 2400 50  0001 C CNN
+F 0 "#PWR06" H 3450 2400 50  0001 C CNN
 F 1 "+5V" H 3450 2690 50  0000 C CNN
 F 2 "" H 3450 2550 50  0001 C CNN
